Commit message: add rx1 gazebo simulation

File: rx1_description/urdf/rx1.urdf (robot description, URDF)
Before this commit: robot rx1, 34 links, 33 joints
Links:
- link base_link: mass 10.0 -> 5.0
- link left_armrot_link: mass None -> 0.3
- link left_elbow_link: mass None -> 0.3
- link left_forearm_link: mass None -> 0.3
- link left_forearm_pitch_link: mass None -> 0.3
- link left_forearm_roll_link: mass None -> 0.3
- link left_forearmrot_link: mass None -> 0.3
- link left_hand_link: mass None -> 0.3
- link left_shoul_base_link: mass 0.05 -> 0.2
- link left_shoul_link: mass None -> 0.3
- link left_shoul_rot_link: mass None -> 0.3
- link left_upper_arm_link: mass None -> 0.3
- link right_armrot_link: mass None -> 0.3
- link right_elbow_link: mass None -> 0.3
- link right_forearm_link: mass None -> 0.3
- link right_forearm_pitch_link: mass None -> 0.3
- link right_forearm_roll_link: mass None -> 0.3
- link right_forearmrot_link: mass None -> 0.3
- link right_hand_link: mass None -> 0.3
- link right_shoul_base_link: mass 0.05 -> 0.2
- link right_shoul_link: mass None -> 0.3
- link right_shoul_rot_link: mass None -> 0.3
- link right_upper_arm_link: mass None -> 0.3
- link torso_link: mass 0.05 -> 0.5
- link torso_pitch_link: mass None -> 0.5
- link torso_roll_link: mass None -> 0.5
- link torso_yaw_link: mass None -> 0.5
Joints:
- joint base2torso_yaw_joint: axis 0 0 1 -> 0.0 0.0 1.0; limit lower=-1.57075 upper=1.57075 effort=50.0 velocity=15 -> lower=-1.57075 upper=1.57075 effort=100.0 velocity=15.0; origin xyz=0 0 0.5825 rpy=0 0 0 -> xyz=0.0 0.0 0.5825 rpy=0.0 0.0 0.0
- joint head_base2left_shoul_base_joint: origin xyz=0 0.12 -0.05 rpy=-1.04706195 0 0 -> xyz=0.0 0.12 -0.05 rpy=-1.04706195 0.0 0.0
- joint head_base2neck_yaw_joint: axis 0 0 1 -> 0.0 0.0 1.0; limit lower=-1.57075 upper=1.57075 effort=50.0 velocity=15 -> lower=-1.57075 upper=1.57075 effort=50.0 velocity=15.0; origin xyz=0 0 0 rpy=0 0 0 -> xyz=0.0 0.0 0.0 rpy=0.0 0.0 0.0
- joint head_base2right_shoul_base_joint: origin xyz=0 -0.12 -0.05 rpy=1.04706195 0 0 -> xyz=0.0 -0.12 -0.05 rpy=1.04706195 0.0 0.0
- joint head_depth_cam_mount2camera_joint: origin xyz=0.05 0 0.03 rpy=0 0 0 -> xyz=0.05 0.0 0.03 rpy=0.0 0.0 0.0
- joint head_depth_cam_mount2left_ear_joint: axis 0 1 0 -> 0.0 1.0 0.0; limit lower=-1.57075 upper=1.57075 effort=50.0 velocity=15 -> lower=-1.57075 upper=1.57075 effort=50.0 velocity=15.0; origin xyz=0 0.065 0.045 rpy=0 0 0 -> xyz=0.0 0.065 0.045 rpy=0.0 0.0 0.0
- joint head_depth_cam_mount2right_ear_joint: axis 0 1 0 -> 0.0 1.0 0.0; limit lower=-1.57075 upper=1.57075 effort=50.0 velocity=15 -> lower=-1.57075 upper=1.57075 effort=50.0 velocity=15.0; origin xyz=0 -0.065 0.045 rpy=0 0 0 -> xyz=0.0 -0.065 0.045 rpy=0.0 0.0 0.0
- joint left_arm2armrot_joint: axis 0 0 1 -> 0.0 0.0 1.0; limit lower=-1.57075 upper=1.57075 effort=50.0 velocity=15 -> lower=-1.57075 upper=1.57075 effort=50.0 velocity=15.0; origin xyz=0 0 -0.0625 rpy=0 0 0 -> xyz=0.0 0.0 -0.0625 rpy=0.0 0.0 0.0
- joint left_armrot2elbow_joint: axis 0 1 0 -> 0.0 1.0 0.0; limit lower=-2.19905 upper=0 effort=50.0 velocity=15 -> lower=-2.19905 upper=0.0 effort=50.0 velocity=15.0; origin xyz=0 0 -0.22 rpy=0 0 0 -> xyz=0.0 0.0 -0.22 rpy=0.0 0.0 0.0
- joint left_elbow2forearm_joint: origin xyz=0 0 -0.045 rpy=0 0 0 -> xyz=0.0 0.0 -0.045 rpy=0.0 0.0 0.0
- joint left_forearm2forearmrot_joint: axis 0 0 1 -> 0.0 0.0 1.0; limit lower=-1.57075 upper=1.57075 effort=50.0 velocity=15 -> lower=-1.57075 upper=1.57075 effort=50.0 velocity=15.0; origin xyz=0 0 -0.045 rpy=0 0 0 -> xyz=0.0 0.0 -0.045 rpy=0.0 0.0 0.0
- joint left_forearm_pitch2forearm_roll_joint: axis 1 0 0 -> 1.0 0.0 0.0; limit lower=-0.785375 upper=0.785375 effort=50.0 velocity=15 -> lower=-0.785375 upper=0.785375 effort=50.0 velocity=15.0; origin xyz=0 0 0 rpy=0 0 0 -> xyz=0.0 0.0 0.0 rpy=0.0 0.0 0.0
- joint left_forearm_roll2hand_joint: origin xyz=0 0 -0.1 rpy=0 0 0 -> xyz=0.0 0.0 -0.1 rpy=0.0 0.0 0.0
- joint left_forearmrot2forearm_pitch_joint: axis 0 1 0 -> 0.0 1.0 0.0; limit lower=-0.785375 upper=0.785375 effort=50.0 velocity=15 -> lower=-0.785375 upper=0.785375 effort=50.0 velocity=15.0; origin xyz=0 0 -0.18 rpy=0 0 0 -> xyz=0.0 0.0 -0.18 rpy=0.0 0.0 0.0
- joint left_shoul2shoul_rot_joint: axis 1 0 0 -> 1.0 0.0 0.0; limit lower=-0.5026400000000001 upper=1.57075 effort=50.0 velocity=15 -> lower=-0.5026400000000001 upper=1.57075 effort=50.0 velocity=15.0; origin xyz=0 0 0.08 rpy=1.04706195 0 0 -> xyz=0.0 0.0 0.08 rpy=1.04706195 0.0 0.0
- joint left_shoul_base2shoul_joint: axis 0 0 1 -> 0.0 0.0 1.0; limit lower=-2.5132000000000003 upper=2.5132000000000003 effort=50.0 velocity=15 -> lower=-2.5132000000000003 upper=2.5132000000000003 effort=50.0 velocity=15.0; origin xyz=0 0 0.075 rpy=0 0 0 -> xyz=0.0 0.0 0.075 rpy=0.0 0.0 0.0
- joint left_shoul_rot2upper_arm_joint: origin xyz=0 0 -0.0625 rpy=0 0 0 -> xyz=0.0 0.0 -0.0625 rpy=0.0 0.0 0.0
- joint neck_pitch2head_depth_cam_mount_joint: axis 1 0 0 -> 1.0 0.0 0.0; limit lower=-1.57075 upper=1.57075 effort=50.0 velocity=15 -> lower=-1.57075 upper=1.57075 effort=50.0 velocity=15.0; origin xyz=-0.01 0 0.1 rpy=0 0 0 -> xyz=-0.01 0.0 0.1 rpy=0.0 0.0 0.0
- joint neck_yaw2pitch_joint: axis 0 1 0 -> 0.0 1.0 0.0; limit lower=-1.57075 upper=1.57075 effort=50.0 velocity=15 -> lower=-1.57075 upper=1.57075 effort=50.0 velocity=15.0; origin xyz=0 0 0.035 rpy=0 0 0 -> xyz=0.0 0.0 0.035 rpy=0.0 0.0 0.0
- joint right_arm2armrot_joint: axis 0 0 1 -> 0.0 0.0 1.0; limit lower=-1.57075 upper=1.57075 effort=50.0 velocity=15 -> lower=-1.57075 upper=1.57075 effort=50.0 velocity=15.0; origin xyz=0 0 -0.0625 rpy=0 0 0 -> xyz=0.0 0.0 -0.0625 rpy=0.0 0.0 0.0
- joint right_armrot2elbow_joint: axis 0 1 0 -> 0.0 1.0 0.0; limit lower=-2.19905 upper=0 effort=50.0 velocity=15 -> lower=-2.19905 upper=0.0 effort=50.0 velocity=15.0; origin xyz=0 0 -0.22 rpy=0 0 0 -> xyz=0.0 0.0 -0.22 rpy=0.0 0.0 0.0
- joint right_elbow2forearm_joint: origin xyz=0 0 -0.045 rpy=0 0 0 -> xyz=0.0 0.0 -0.045 rpy=0.0 0.0 0.0
- joint right_forearm2forearmrot_joint: axis 0 0 1 -> 0.0 0.0 1.0; limit lower=-1.57075 upper=1.57075 effort=50.0 velocity=15 -> lower=-1.57075 upper=1.57075 effort=50.0 velocity=15.0; origin xyz=0 0 -0.045 rpy=0 0 0 -> xyz=0.0 0.0 -0.045 rpy=0.0 0.0 0.0
- joint right_forearm_pitch2forearm_roll_joint: axis 1 0 0 -> 1.0 0.0 0.0; limit lower=-0.785375 upper=0.785375 effort=50.0 velocity=15 -> lower=-0.785375 upper=0.785375 effort=50.0 velocity=15.0; origin xyz=0 0 0 rpy=0 0 0 -> xyz=0.0 0.0 0.0 rpy=0.0 0.0 0.0
- joint right_forearm_roll2hand_joint: origin xyz=0 0 -0.1 rpy=0 0 0 -> xyz=0.0 0.0 -0.1 rpy=0.0 0.0 0.0
- joint right_forearmrot2forearm_pitch_joint: axis 0 1 0 -> 0.0 1.0 0.0; limit lower=-0.785375 upper=0.785375 effort=50.0 velocity=15 -> lower=-0.785375 upper=0.785375 effort=50.0 velocity=15.0; origin xyz=0 0 -0.18 rpy=0 0 0 -> xyz=0.0 0.0 -0.18 rpy=0.0 0.0 0.0
- joint right_shoul2shoul_rot_joint: axis 1 0 0 -> 1.0 0.0 0.0; limit lower=-1.57075 upper=0.5026400000000001 effort=50.0 velocity=15 -> lower=-1.57075 upper=0.5026400000000001 effort=50.0 velocity=15.0; origin xyz=0 0 0.08 rpy=-1.04706195 0 0 -> xyz=0.0 0.0 0.08 rpy=-1.04706195 0.0 0.0
- joint right_shoul_base2shoul_joint: axis 0 0 1 -> 0.0 0.0 1.0; limit lower=-2.5132000000000003 upper=2.5132000000000003 effort=50.0 velocity=15 -> lower=-2.5132000000000003 upper=2.5132000000000003 effort=50.0 velocity=15.0; origin xyz=0 0 0.075 rpy=0 0 0 -> xyz=0.0 0.0 0.075 rpy=0.0 0.0 0.0
- joint right_shoul_rot2upper_arm_joint: origin xyz=0 0 -0.0625 rpy=0 0 0 -> xyz=0.0 0.0 -0.0625 rpy=0.0 0.0 0.0
- joint torso2head_base_joint: origin xyz=0 0 0.21 rpy=0 0 0 -> xyz=0.0 0.0 0.21 rpy=0.0 0.0 0.0
- joint torso_pitch2roll_joint: axis 1 0 0 -> 1.0 0.0 0.0; limit lower=-0.785375 upper=0.785375 effort=50.0 velocity=15 -> lower=-0.785375 upper=0.785375 effort=100.0 velocity=15.0; origin xyz=0 0 0 rpy=0 0 0 -> xyz=0.0 0.0 0.0 rpy=0.0 0.0 0.0
- joint torso_roll2torso_joint: origin xyz=0 0 0.08 rpy=0 0 0 -> xyz=0.0 0.0 0.08 rpy=0.0 0.0 0.0
- joint torso_yaw2pitch_joint: axis 0 1 0 -> 0.0 1.0 0.0; limit lower=-0.785375 upper=0.785375 effort=50.0 velocity=15 -> lower=-0.785375 upper=0.785375 effort=100.0 velocity=15.0; origin xyz=0 0 0.15 rpy=0 0 0 -> xyz=0.0 0.0 0.15 rpy=0.0 0.0 0.0

File: rx1_description/urdf/rx1.urdf.xacro (robot description, xacro)
@@ -22,5 +22,5 @@
     <link name="base_link">
         <inertial>
-            <mass value="10.0" />
+            <mass value="5.0" />
             <inertia ixx="0.1" ixy="0.0" ixz="0.0" iyy="0.04" iyz="0.0" izz="0.2" />
         </inertial>
@@ -39,4 +39,8 @@
     <!--                            TORSO START                         -->
     <link name="torso_yaw_link">
+        <inertial>
+            <mass value="0.5" />
+            <inertia ixx="1.0" ixy="0.0" ixz="0.0" iyy="1.0" iyz="0.0" izz="1.0" />
+        </inertial>
         <visual>
             <geometry>
@@ -61,4 +65,8 @@
     </joint>
     <link name="torso_pitch_link">
+        <inertial>
+            <mass value="0.5" />
+            <inertia ixx="1.0" ixy="0.0" ixz="0.0" iyy="1.0" iyz="0.0" izz="1.0" />
+        </inertial>
         <visual>
             <geometry>
@@ -83,4 +91,8 @@
     </joint>
     <link name="torso_roll_link">
+        <inertial>
+            <mass value="0.5" />
+            <inertia ixx="1.0" ixy="0.0" ixz="0.0" iyy="1.0" iyz="0.0" izz="1.0" />
+        </inertial>
         <visual>
             <geometry>
@@ -106,5 +118,5 @@
     <link name="torso_link">
         <inertial>
-            <mass value="0.05" />
+            <mass value="0.5" />
             <inertia ixx="4.16666667e-06" ixy="0.0" ixz="0.0" iyy="6.6666666667e-6" iyz="0.0" izz="04.16666667e-06" />
         </inertial>
@@ -315,5 +327,5 @@
         <link name="${prefix}_shoul_base_link">
             <inertial>
-                <mass value="0.05" />
+                <mass value="0.2" />
                 <inertia ixx="4.16666667e-06" ixy="0.0" ixz="0.0" iyy="6.6666666667e-6" iyz="0.0" izz="04.16666667e-06" />
             </inertial>
@@ -338,4 +350,8 @@
         </joint>
         <link name="${prefix}_shoul_link">
+            <inertial>
+                <mass value="0.3" />
+                <inertia ixx="1.0" ixy="0.0" ixz="0.0" iyy="1.0" iyz="0.0" izz="1.0" />
+            </inertial>
             <visual>
                 <geometry>
@@ -360,4 +376,8 @@
         </joint>
         <link name="${prefix}_shoul_rot_link">
+            <inertial>
+                <mass value="0.3" />
+                <inertia ixx="1.0" ixy="0.0" ixz="0.0" iyy="1.0" iyz="0.0" izz="1.0" />
+            </inertial>
             <visual>
                 <geometry>
@@ -387,5 +407,9 @@
         </joint>
         <link name="${prefix}_upper_arm_link">
-            <visual>
+           <inertial>
+                <mass value="0.3" />
+                <inertia ixx="1.0" ixy="0.0" ixz="0.0" iyy="1.0" iyz="0.0" izz="1.0" />
+           </inertial>
+           <visual>
                 <geometry>
                     <!--cylinder length="0.085" radius="0.015" /-->
@@ -409,4 +433,8 @@
         </joint>
         <link name="${prefix}_armrot_link">
+            <inertial>
+                <mass value="0.3" />
+                <inertia ixx="1.0" ixy="0.0" ixz="0.0" iyy="1.0" iyz="0.0" izz="1.0" />
+            </inertial>
             <visual>
                 <geometry>
@@ -432,4 +460,8 @@
         </joint>
         <link name="${prefix}_elbow_link">
+            <inertial>
+                <mass value="0.3" />
+                <inertia ixx="1.0" ixy="0.0" ixz="0.0" iyy="1.0" iyz="0.0" izz="1.0" />
+            </inertial>
             <visual>
                 <geometry>
@@ -454,4 +486,8 @@
         </joint>
         <link name="${prefix}_forearm_link">
+            <inertial>
+                <mass value="0.3" />
+                <inertia ixx="1.0" ixy="0.0" ixz="0.0" iyy="1.0" iyz="0.0" izz="1.0" />
+            </inertial>
             <visual>
                 <geometry>
@@ -474,4 +510,8 @@
         </joint>
         <link name="${prefix}_forearmrot_link">
+            <inertial>
+                <mass value="0.3" />
+                <inertia ixx="1.0" ixy="0.0" ixz="0.0" iyy="1.0" iyz="0.0" izz="1.0" />
+            </inertial>
             <visual>
                 <geometry>
@@ -497,4 +537,8 @@
         </joint>
         <link name="${prefix}_forearm_pitch_link">
+            <inertial>
+                <mass value="0.3" />
+                <inertia ixx="1.0" ixy="0.0" ixz="0.0" iyy="1.0" iyz="0.0" izz="1.0" />
+            </inertial>
             <visual>
                 <geometry>
@@ -519,4 +563,8 @@
         </joint>
         <link name="${prefix}_forearm_roll_link">
+            <inertial>
+                <mass value="0.3" />
+                <inertia ixx="1.0" ixy="0.0" ixz="0.0" iyy="1.0" iyz="0.0" izz="1.0" />
+            </inertial>
             <visual>
                 <geometry>
@@ -541,4 +589,8 @@
         </joint>
         <link name="${prefix}_hand_link">
+            <inertial>
+                <mass value="0.3" />
+                <inertia ixx="1.0" ixy="0.0" ixz="0.0" iyy="1.0" iyz="0.0" izz="1.0" />
+            </inertial>
             <visual>
                 <geometry>
