Commit message: add torso and head urdf

File: rx1_description/urdf/rx1.urdf.xacro (robot description, xacro)
@@ -27,14 +27,17 @@
         <visual>
             <geometry>
-                <box size="0.02 0.02 0.5" />
-            </geometry>
-            <material name="white"/>
-        </visual>
-        <collision>
-            <geometry>
-                <box size="0.02 0.02 0.5" />
-            </geometry>
-        </collision>
-    </link>
+                <!--box size="0.02 0.02 0.5" /-->
+                <mesh filename="package://rx1_description/meshes/base_link.stl"/>
+            </geometry>
+            <material name="white"/>
+        </visual>
+        <collision>
+            <geometry>
+                <!--box size="0.02 0.02 0.5" /-->
+                <mesh filename="package://rx1_description/meshes/base_link.stl"/>
+            </geometry>
+        </collision>
+    </link>
+<!--
     <link name="camera_link">
         <inertial>
@@ -75,4 +78,72 @@
         <child link="camera_color_optical_frame" />
     </joint>
+-->
+    <!--                            TORSO START                         -->
+    <link name="torso_yaw_link">
+        <visual>
+            <geometry>
+                <mesh filename="package://rx1_description/meshes/torso_yaw_link.stl"/>
+            </geometry>
+            <origin rpy="0 0 0" xyz="0 0 0"/>
+            <material name="white"/>
+        </visual>
+        <collision>
+            <geometry>
+                <mesh filename="package://rx1_description/meshes/torso_yaw_link.stl"/>
+            </geometry>
+            <origin rpy="0 0 0" xyz="0 0 0"/>
+        </collision>
+    </link>
+    <joint name="base2torso_yaw_joint" type="revolute">
+        <axis xyz="0 0 1" />
+        <limit effort="${motor_torque}" lower="${-0.5*pi}" upper="${0.5*pi}" velocity="${motor_vec}"/>
+        <origin xyz="0 0 0.5825" rpy="0 0 0" />
+        <parent link="base_link" />
+        <child link="torso_yaw_link" />
+    </joint>
+    <link name="torso_pitch_link">
+        <visual>
+            <geometry>
+                <cylinder length="0.03" radius="0.015" />
+            </geometry>
+            <origin rpy="${0.5*pi} 0 0" xyz="0 0 0"/>
+            <material name="blue"/>
+        </visual>
+        <collision>
+            <geometry>
+                <cylinder length="0.03" radius="0.01" />
+            </geometry>
+            <origin rpy="${0.5*pi} 0 0" xyz="0 0 0"/>
+        </collision>
+    </link>
+    <joint name="torso_yaw2pitch_joint" type="revolute">
+        <axis xyz="0 1 0" />
+        <limit effort="${motor_torque}" lower="${-0.25*pi}" upper="${0.25*pi}" velocity="${motor_vec}"/>
+        <origin xyz="0 0 0.15" rpy="0 0 0" />
+        <parent link="torso_yaw_link" />
+        <child link="torso_pitch_link" />
+    </joint>
+    <link name="torso_roll_link">
+        <visual>
+            <geometry>
+                <cylinder length="0.03" radius="0.015" />
+            </geometry>
+            <origin rpy="0 ${0.5*pi} 0" xyz="0 0 0"/>
+            <material name="red"/>
+        </visual>
+        <collision>
+            <geometry>
+                <cylinder length="0.03" radius="0.01" />
+            </geometry>
+            <origin rpy="0 ${0.5*pi} 0" xyz="0 0 0"/>
+        </collision>
+    </link>
+    <joint name="torso_pitch2roll_joint" type="revolute">
+        <axis xyz="1 0 0" />
+        <limit effort="${motor_torque}" lower="${-0.25*pi}" upper="${0.25*pi}" velocity="${motor_vec}"/>
+        <origin xyz="0 0 0" rpy="0 0 0" />
+        <parent link="torso_pitch_link" />
+        <child link="torso_roll_link" />
+    </joint>
     <link name="torso_link">
         <inertial>
@@ -83,21 +154,180 @@
             <geometry>
                 <!--box size="0.03 0.12 0.02" /-->
-                <mesh filename="package://rx1_description/meshes/torso_link_v2.stl"/>
-            </geometry>
-            <origin rpy="0 0 0" xyz="0 0 0"/>
-            <material name="white"/>
-        </visual>
-        <collision>
-            <geometry>
-                <box size="0.03 0.12 0.02" />
-            </geometry>
-            <origin rpy="0 0 0" xyz="0 0 0"/>
-        </collision>
-    </link>
-    <joint name="base2torso_joint" type="fixed">
-        <origin xyz="0 0 0.26" rpy="0 0 0" />
-        <parent link="base_link" />
+                <mesh filename="package://rx1_description/meshes/torso_link.stl"/>
+            </geometry>
+            <origin rpy="0 0 0" xyz="0 0 0"/>
+            <material name="white"/>
+        </visual>
+        <collision>
+            <geometry>
+                <!--box size="0.03 0.12 0.02" /-->
+                <mesh filename="package://rx1_description/meshes/torso_link.stl"/>
+            </geometry>
+            <origin rpy="0 0 0" xyz="0 0 0"/>
+        </collision>
+    </link>
+    <joint name="torso_roll2torso_joint" type="fixed">
+        <origin xyz="0 0 0.08" rpy="0 0 0" />
+        <parent link="torso_roll_link" />
         <child link="torso_link" />
     </joint>
+    <!--                            TORSO END                         -->
+    <!--                            HEAD START                        -->
+    <link name="head_base_link">
+        <inertial>
+            <mass value="0.05" />
+            <inertia ixx="4.16666667e-06" ixy="0.0" ixz="0.0" iyy="6.6666666667e-6" iyz="0.0" izz="04.16666667e-06" />
+        </inertial>
+        <visual>
+            <geometry>
+                <mesh filename="package://rx1_description/meshes/head/head_base_link.stl"/>
+            </geometry>
+            <origin rpy="0 0 0" xyz="0 0 0"/>
+            <material name="white"/>
+        </visual>
+        <collision>
+            <geometry>
+                <mesh filename="package://rx1_description/meshes/head/head_base_link.stl"/>
+            </geometry>
+            <origin rpy="0 0 0" xyz="0 0 0"/>
+        </collision>
+    </link>
+    <joint name="torso2head_base_joint" type="fixed">
+        <origin xyz="0 0 0.21" rpy="0 0 0" />
+        <parent link="torso_link" />
+        <child link="head_base_link" />
+    </joint>
+    <link name="neck_yaw_link">
+        <inertial>
+            <mass value="0.05" />
+            <inertia ixx="4.16666667e-06" ixy="0.0" ixz="0.0" iyy="6.6666666667e-6" iyz="0.0" izz="04.16666667e-06" />
+        </inertial>
+        <visual>
+            <geometry>
+                <mesh filename="package://rx1_description/meshes/head/neck_yaw_link.stl"/>
+            </geometry>
+            <origin rpy="0 0 0" xyz="0 0 0"/>
+            <material name="white"/>
+        </visual>
+        <collision>
+            <geometry>
+                <mesh filename="package://rx1_description/meshes/head/neck_yaw_link.stl"/>
+            </geometry>
+            <origin rpy="0 0 0" xyz="0 0 0"/>
+        </collision>
+    </link>
+    <joint name="head_base2neck_yaw_joint" type="revolute">
+        <axis xyz="0 0 1" />
+        <limit effort="${motor_torque}" lower="${-0.5*pi}" upper="${0.5*pi}" velocity="${motor_vec}"/>
+        <origin xyz="0 0 0" rpy="0 0 0" />
+        <parent link="head_base_link" />
+        <child link="neck_yaw_link" />
+    </joint>
+    <link name="neck_pitch_link">
+        <inertial>
+            <mass value="0.05" />
+            <inertia ixx="4.16666667e-06" ixy="0.0" ixz="0.0" iyy="6.6666666667e-6" iyz="0.0" izz="04.16666667e-06" />
+        </inertial>
+        <visual>
+            <geometry>
+                <mesh filename="package://rx1_description/meshes/head/neck_pitch_link.stl"/>
+            </geometry>
+            <origin rpy="0 0 0" xyz="0 0 0"/>
+            <material name="white"/>
+        </visual>
+        <collision>
+            <geometry>
+                <mesh filename="package://rx1_description/meshes/head/neck_pitch_link.stl"/>
+            </geometry>
+            <origin rpy="0 0 0" xyz="0 0 0"/>
+        </collision>
+    </link>
+    <joint name="neck_yaw2pitch_joint" type="revolute">
+        <axis xyz="0 1 0" />
+        <limit effort="${motor_torque}" lower="${-0.5*pi}" upper="${0.5*pi}" velocity="${motor_vec}"/>
+        <origin xyz="0 0 0.035" rpy="0 0 0" />
+        <parent link="neck_yaw_link" />
+        <child link="neck_pitch_link" />
+    </joint>
+    <link name="head_depth_cam_mount_link">
+        <inertial>
+            <mass value="0.05" />
+            <inertia ixx="4.16666667e-06" ixy="0.0" ixz="0.0" iyy="6.6666666667e-6" iyz="0.0" izz="04.16666667e-06" />
+        </inertial>
+        <visual>
+            <geometry>
+                <mesh filename="package://rx1_description/meshes/head/head_depth_cam_mount_link.stl"/>
+            </geometry>
+            <origin rpy="0 0 0" xyz="0 0 0"/>
+            <material name="white"/>
+        </visual>
+        <collision>
+            <geometry>
+                <mesh filename="package://rx1_description/meshes/head/head_depth_cam_mount_link.stl"/>
+            </geometry>
+            <origin rpy="0 0 0" xyz="0 0 0"/>
+        </collision>
+    </link>
+    <joint name="neck_pitch2head_depth_cam_mount_joint" type="revolute">
+        <axis xyz="1 0 0" />
+        <limit effort="${motor_torque}" lower="${-0.5*pi}" upper="${0.5*pi}" velocity="${motor_vec}"/>
+        <origin xyz="-0.01 0 0.1" rpy="0 0 0" />
+        <parent link="neck_pitch_link" />
+        <child link="head_depth_cam_mount_link" />
+    </joint>
+    <link name="right_ear_link">
+        <inertial>
+            <mass value="0.05" />
+            <inertia ixx="4.16666667e-06" ixy="0.0" ixz="0.0" iyy="6.6666666667e-6" iyz="0.0" izz="04.16666667e-06" />
+        </inertial>
+        <visual>
+            <geometry>
+                <mesh filename="package://rx1_description/meshes/head/right_ear_link.stl"/>
+            </geometry>
+            <origin rpy="0 0 0" xyz="0 0 0"/>
+            <material name="white"/>
+        </visual>
+        <collision>
+            <geometry>
+                <mesh filename="package://rx1_description/meshes/head/right_ear_link.stl"/>
+            </geometry>
+            <origin rpy="0 0 0" xyz="0 0 0"/>
+        </collision>
+    </link>
+    <joint name="head_depth_cam_mount2right_ear_joint" type="revolute">
+        <axis xyz="0 1 0" />
+        <limit effort="${motor_torque}" lower="${-0.5*pi}" upper="${0.5*pi}" velocity="${motor_vec}"/>
+        <origin xyz="0 -0.065 0.045" rpy="0 0 0" />
+        <parent link="head_depth_cam_mount_link" />
+        <child link="right_ear_link" />
+    </joint>
+    <link name="left_ear_link">
+        <inertial>
+            <mass value="0.05" />
+            <inertia ixx="4.16666667e-06" ixy="0.0" ixz="0.0" iyy="6.6666666667e-6" iyz="0.0" izz="04.16666667e-06" />
+        </inertial>
+        <visual>
+            <geometry>
+                <mesh filename="package://rx1_description/meshes/head/left_ear_link.stl"/>
+            </geometry>
+            <origin rpy="0 0 0" xyz="0 0 0"/>
+            <material name="white"/>
+        </visual>
+        <collision>
+            <geometry>
+                <mesh filename="package://rx1_description/meshes/head/left_ear_link.stl"/>
+            </geometry>
+            <origin rpy="0 0 0" xyz="0 0 0"/>
+        </collision>
+    </link>
+    <joint name="head_depth_cam_mount2left_ear_joint" type="revolute">
+        <axis xyz="0 1 0" />
+        <limit effort="${motor_torque}" lower="${-0.5*pi}" upper="${0.5*pi}" velocity="${motor_vec}"/>
+        <origin xyz="0 0.065 0.045" rpy="0 0 0" />
+        <parent link="head_depth_cam_mount_link" />
+        <child link="left_ear_link" />
+    </joint>
+    <!--                            HEAD END                           -->
+    <!--                            ARM START                          -->
     <xacro:macro name="arm" params="prefix side">
         <link name="${prefix}_shoul_base_link">
@@ -121,5 +351,5 @@
         </link>
         <joint name="torso2${prefix}_shoul_base_joint" type="fixed">
-            <origin xyz="0 ${-0.12*side} -0.04" rpy="${0.3333*pi*side} 0 0" />
+            <origin xyz="0 ${-0.12*side} 0.16" rpy="${0.3333*pi*side} 0 0" />
             <parent link="torso_link" />
             <child link="${prefix}_shoul_base_link" />
@@ -353,3 +583,4 @@
     <xacro:arm prefix="right" side="1" />
     <xacro:arm prefix="left" side="-1" />
+    <!--                            ARM END                             -->
 </robot>

Commit message: update motor node for dual arm, head, and torso

File: rx1_description/urdf/rx1.urdf.xacro (robot description, xacro)
@@ -276,4 +276,28 @@
         <child link="head_depth_cam_mount_link" />
     </joint>
+    <link name="camera_link">
+        <inertial>
+            <mass value="0.05" />
+            <inertia ixx="4.16666667e-06" ixy="0.0" ixz="0.0" iyy="6.6666666667e-6" iyz="0.0" izz="04.16666667e-06" />
+        </inertial>
+        <visual>
+            <geometry>
+                <box size="0.01 0.01 0.01" />
+            </geometry>
+            <origin rpy="0 0 0" xyz="0 0 0"/>
+            <material name="white"/>
+        </visual>
+        <collision>
+            <geometry>
+                <box size="0.01 0.01 0.01" />
+            </geometry>
+            <origin rpy="0 0 0" xyz="0 0 0"/>
+        </collision>
+    </link>
+    <joint name="head_depth_cam_mount2camera_joint" type="fixed">
+        <origin xyz="0.05 0 0.03" rpy="0 0 0" />
+        <parent link="head_depth_cam_mount_link" />
+        <child link="camera_link" />
+    </joint>
     <link name="right_ear_link">
         <inertial>

Commit message: ik update for dual arm

File: rx1_description/urdf/rx1.urdf.xacro (robot description, xacro)
@@ -374,7 +374,7 @@
             </collision>
         </link>
-        <joint name="torso2${prefix}_shoul_base_joint" type="fixed">
-            <origin xyz="0 ${-0.12*side} 0.16" rpy="${0.3333*pi*side} 0 0" />
-            <parent link="torso_link" />
+        <joint name="head_base2${prefix}_shoul_base_joint" type="fixed">
+            <origin xyz="0 ${-0.12*side} -0.05" rpy="${0.3333*pi*side} 0 0" />
+            <parent link="head_base_link" />
             <child link="${prefix}_shoul_base_link" />
         </joint>

Commit message: urdf, motor and ik code cleanup

File: rx1_description/urdf/rx1.urdf.xacro (robot description, xacro)
@@ -1,3 +1,4 @@
 <?xml version="1.0"?>
+<!--Note that the inertia values are placeholder and need to be updated for proper physics simulation-->
 <robot name="rx1" xmlns:xacro="http://ros.org/wiki/xacro">
     <xacro:property name="pi" value="3.1415" />
@@ -23,9 +24,7 @@
             <mass value="10.0" />
             <inertia ixx="0.1" ixy="0.0" ixz="0.0" iyy="0.04" iyz="0.0" izz="0.2" />
-            <!--inertia ixx="1" ixy="0.0" ixz="0.0" iyy="1" iyz="0.0" izz="1" /-->
-        </inertial>
-        <visual>
-            <geometry>
-                <!--box size="0.02 0.02 0.5" /-->
+        </inertial>
+        <visual>
+            <geometry>
                 <mesh filename="package://rx1_description/meshes/base_link.stl"/>
             </geometry>
@@ -34,49 +33,8 @@
         <collision>
             <geometry>
-                <!--box size="0.02 0.02 0.5" /-->
                 <mesh filename="package://rx1_description/meshes/base_link.stl"/>
             </geometry>
         </collision>
     </link>
-<!--
-    <link name="camera_link">
-        <inertial>
-            <mass value="0.05" />
-            <inertia ixx="4.16666667e-06" ixy="0.0" ixz="0.0" iyy="6.6666666667e-6" iyz="0.0" izz="04.16666667e-06" />
-        </inertial>
-        <visual>
-            <geometry>
-                <box size="0.02 0.08 0.02" />
-            </geometry>
-            <origin rpy="0 0 0" xyz="0 0 0"/>
-            <material name="white"/>
-        </visual>
-        <collision>
-            <geometry>
-                <box size="0.03 0.12 0.02" />
-            </geometry>
-            <origin rpy="0 0 0" xyz="0 0 0"/>
-        </collision>
-    </link>
-    <joint name="base2camera_joint" type="fixed">
-        <origin xyz="0 0 0.40" rpy="0 0.5 0" />
-        <parent link="base_link" />
-        <child link="camera_link" />
-    </joint>
-    <link name="camera_color_optical_frame">
-        <visual>
-            <geometry>
-                <box size="0.01 0.01 0.01" />
-            </geometry>
-            <origin rpy="0 0 0" xyz="0 0 0"/>
-            <material name="white"/>
-        </visual>
-    </link>
-    <joint name="camera2camera_joint" type="fixed">
-        <origin xyz="0 0 0" rpy="-1.57 0 -1.57" />
-        <parent link="camera_link" />
-        <child link="camera_color_optical_frame" />
-    </joint>
--->
     <!--                            TORSO START                         -->
     <link name="torso_yaw_link">
@@ -418,5 +376,4 @@
         <joint name="${prefix}_shoul2shoul_rot_joint" type="revolute">
             <axis xyz="1 0 0" />
-            <!--limit effort="${motor_torque}" lower="${-0.5*pi}" upper="${0.16*pi}" velocity="${motor_vec}"/-->
             <xacro:if value="${prefix == 'right'}">
                 <limit effort="${motor_torque}" lower="${-0.5*pi}" upper="${0.16*pi}" velocity="${motor_vec}"/>
