Commit message: gazebo simulation physics tuning and add controller testing gui

File: rx1_description/urdf/rx1.urdf.xacro (robot description, xacro)
@@ -40,5 +40,5 @@
     <link name="torso_yaw_link">
         <inertial>
-            <mass value="0.5" />
+            <mass value="5.0" />
             <inertia ixx="1.0" ixy="0.0" ixz="0.0" iyy="1.0" iyz="0.0" izz="1.0" />
         </inertial>
@@ -60,4 +60,5 @@
         <axis xyz="0 0 1" />
         <limit effort="${motor_torque}" lower="${-0.5*pi}" upper="${0.5*pi}" velocity="${motor_vec}"/>
+        <dynamics damping="0.5" friction="5.0" />
         <origin xyz="0 0 0.5825" rpy="0 0 0" />
         <parent link="base_link" />
@@ -86,4 +87,5 @@
         <axis xyz="0 1 0" />
         <limit effort="${motor_torque}" lower="${-0.25*pi}" upper="${0.25*pi}" velocity="${motor_vec}"/>
+        <dynamics damping="5" friction="10.0" />
         <origin xyz="0 0 0.15" rpy="0 0 0" />
         <parent link="torso_yaw_link" />
@@ -112,4 +114,5 @@
         <axis xyz="1 0 0" />
         <limit effort="${motor_torque}" lower="${-0.25*pi}" upper="${0.25*pi}" velocity="${motor_vec}"/>
+        <dynamics damping="5" friction="10" />
         <origin xyz="0 0 0" rpy="0 0 0" />
         <parent link="torso_pitch_link" />
@@ -118,5 +121,5 @@
     <link name="torso_link">
         <inertial>
-            <mass value="0.5" />
+            <mass value="2" />
             <inertia ixx="4.16666667e-06" ixy="0.0" ixz="0.0" iyy="6.6666666667e-6" iyz="0.0" izz="04.16666667e-06" />
         </inertial>
@@ -190,4 +193,5 @@
         <axis xyz="0 0 1" />
         <limit effort="${motor_torque}" lower="${-0.5*pi}" upper="${0.5*pi}" velocity="${motor_vec}"/>
+        <dynamics damping="0.5" friction="0.1" />
         <origin xyz="0 0 0" rpy="0 0 0" />
         <parent link="head_base_link" />
@@ -216,4 +220,5 @@
         <axis xyz="0 1 0" />
         <limit effort="${motor_torque}" lower="${-0.5*pi}" upper="${0.5*pi}" velocity="${motor_vec}"/>
+        <dynamics damping="0.5" friction="0.1" />
         <origin xyz="0 0 0.035" rpy="0 0 0" />
         <parent link="neck_yaw_link" />
@@ -242,4 +247,5 @@
         <axis xyz="1 0 0" />
         <limit effort="${motor_torque}" lower="${-0.5*pi}" upper="${0.5*pi}" velocity="${motor_vec}"/>
+        <dynamics damping="0.1" friction="0.0" />
         <origin xyz="-0.01 0 0.1" rpy="0 0 0" />
         <parent link="neck_pitch_link" />
@@ -292,4 +298,5 @@
         <axis xyz="0 1 0" />
         <limit effort="${motor_torque}" lower="${-0.5*pi}" upper="${0.5*pi}" velocity="${motor_vec}"/>
+        <dynamics damping="0.1" friction="0.0" />
         <origin xyz="0 -0.065 0.045" rpy="0 0 0" />
         <parent link="head_depth_cam_mount_link" />
@@ -318,4 +325,5 @@
         <axis xyz="0 1 0" />
         <limit effort="${motor_torque}" lower="${-0.5*pi}" upper="${0.5*pi}" velocity="${motor_vec}"/>
+        <dynamics damping="0.1" friction="0.0" />
         <origin xyz="0 0.065 0.045" rpy="0 0 0" />
         <parent link="head_depth_cam_mount_link" />
@@ -351,5 +359,5 @@
         <link name="${prefix}_shoul_link">
             <inertial>
-                <mass value="0.3" />
+                <mass value="0.2" />
                 <inertia ixx="1.0" ixy="0.0" ixz="0.0" iyy="1.0" iyz="0.0" izz="1.0" />
             </inertial>
@@ -371,4 +379,5 @@
             <axis xyz="0 0 1" />
             <limit effort="${motor_torque}" lower="${-0.8*pi}" upper="${0.8*pi}" velocity="${motor_vec}"/>
+            <dynamics damping="0.5" friction="0.1" />
             <origin xyz="0 0 0.075" rpy="0 0 0" />
             <parent link="${prefix}_shoul_base_link" />
@@ -377,5 +386,5 @@
         <link name="${prefix}_shoul_rot_link">
             <inertial>
-                <mass value="0.3" />
+                <mass value="0.2" />
                 <inertia ixx="1.0" ixy="0.0" ixz="0.0" iyy="1.0" iyz="0.0" izz="1.0" />
             </inertial>
@@ -398,7 +407,9 @@
             <xacro:if value="${prefix == 'right'}">
                 <limit effort="${motor_torque}" lower="${-0.5*pi}" upper="${0.16*pi}" velocity="${motor_vec}"/>
+                <dynamics damping="0.5" friction="0.1" />
             </xacro:if>
             <xacro:if value="${prefix == 'left'}">
                 <limit effort="${motor_torque}" lower="${-0.16*pi}" upper="${0.5*pi}" velocity="${motor_vec}"/>
+                <dynamics damping="0.5" friction="0.1" />
             </xacro:if>
             <origin xyz="0 0 0.08" rpy="${-0.3333*pi*side} 0 0" />
@@ -408,5 +419,5 @@
         <link name="${prefix}_upper_arm_link">
            <inertial>
-                <mass value="0.3" />
+                <mass value="0.1" />
                 <inertia ixx="1.0" ixy="0.0" ixz="0.0" iyy="1.0" iyz="0.0" izz="1.0" />
            </inertial>
@@ -434,5 +445,5 @@
         <link name="${prefix}_armrot_link">
             <inertial>
-                <mass value="0.3" />
+                <mass value="0.1" />
                 <inertia ixx="1.0" ixy="0.0" ixz="0.0" iyy="1.0" iyz="0.0" izz="1.0" />
             </inertial>
@@ -455,4 +466,5 @@
             <axis xyz="0 0 1" />
             <limit effort="${motor_torque}" lower="${-0.5*pi}" upper="${0.5*pi}" velocity="${motor_vec}"/>
+            <dynamics damping="0.1" friction="0.1" />
             <origin xyz="0 0 -0.0625" rpy="0 0 0" />
             <parent link="${prefix}_upper_arm_link" />
@@ -461,5 +473,5 @@
         <link name="${prefix}_elbow_link">
             <inertial>
-                <mass value="0.3" />
+                <mass value="0.1" />
                 <inertia ixx="1.0" ixy="0.0" ixz="0.0" iyy="1.0" iyz="0.0" izz="1.0" />
             </inertial>
@@ -481,4 +493,5 @@
             <axis xyz="0 1 0" />
             <limit effort="${motor_torque}" lower="${-0.7*pi}" upper="0" velocity="${motor_vec}"/>
+            <dynamics damping="0.1" friction="0.1" />
             <origin xyz="0 0 -0.22" rpy="0 0 0" />
             <parent link="${prefix}_armrot_link" />
@@ -487,5 +500,5 @@
         <link name="${prefix}_forearm_link">
             <inertial>
-                <mass value="0.3" />
+                <mass value="0.1" />
                 <inertia ixx="1.0" ixy="0.0" ixz="0.0" iyy="1.0" iyz="0.0" izz="1.0" />
             </inertial>
@@ -511,5 +524,5 @@
         <link name="${prefix}_forearmrot_link">
             <inertial>
-                <mass value="0.3" />
+                <mass value="0.1" />
                 <inertia ixx="1.0" ixy="0.0" ixz="0.0" iyy="1.0" iyz="0.0" izz="1.0" />
             </inertial>
@@ -532,4 +545,5 @@
             <axis xyz="0 0 1" />
             <limit effort="${motor_torque}" lower="${-0.5*pi}" upper="${0.5*pi}" velocity="${motor_vec}"/>
+            <dynamics damping="0.1" friction="0.1" />
             <origin xyz="0 0 -0.045" rpy="0 0 0" />
             <parent link="${prefix}_forearm_link" />
@@ -538,5 +552,5 @@
         <link name="${prefix}_forearm_pitch_link">
             <inertial>
-                <mass value="0.3" />
+                <mass value="0.1" />
                 <inertia ixx="1.0" ixy="0.0" ixz="0.0" iyy="1.0" iyz="0.0" izz="1.0" />
             </inertial>
@@ -558,4 +572,5 @@
             <axis xyz="0 1 0" />
             <limit effort="${motor_torque}" lower="${-0.25*pi}" upper="${0.25*pi}" velocity="${motor_vec}"/>
+            <dynamics damping="0.1" friction="0.1" />
             <origin xyz="0 0 -0.18" rpy="0 0 0" />
             <parent link="${prefix}_forearmrot_link" />
@@ -564,5 +579,5 @@
         <link name="${prefix}_forearm_roll_link">
             <inertial>
-                <mass value="0.3" />
+                <mass value="0.1" />
                 <inertia ixx="1.0" ixy="0.0" ixz="0.0" iyy="1.0" iyz="0.0" izz="1.0" />
             </inertial>
@@ -584,4 +599,5 @@
             <axis xyz="1 0 0" />
             <limit effort="${motor_torque}" lower="${-0.25*pi}" upper="${0.25*pi}" velocity="${motor_vec}"/>
+            <dynamics damping="0.1" friction="0.1" />
             <origin xyz="0 0 0" rpy="0 0 0" />
             <parent link="${prefix}_forearm_pitch_link" />
@@ -590,5 +606,5 @@
         <link name="${prefix}_hand_link">
             <inertial>
-                <mass value="0.3" />
+                <mass value="0.1" />
                 <inertia ixx="1.0" ixy="0.0" ixz="0.0" iyy="1.0" iyz="0.0" izz="1.0" />
             </inertial>
