Commit message: gazebo simulation update and add readme

File: rx1_description/urdf/rx1.gazebo.urdf (robot description, URDF)
Before this commit: robot robotic_arm, 1 links, 1 joints
Joints:
- joint world_base_joint: origin (none) -> xyz=0.0 0.0 0.2 rpy=0.0 0.0 0.0

File: rx1_description/urdf/rx1.urdf (robot description, URDF)
Before this commit: robot rx1, 34 links, 33 joints
Links:
- link torso_link: mass 2.0 -> 1.0

File: rx1_description/urdf/rx1.urdf.xacro (robot description, xacro)
@@ -87,5 +87,5 @@
         <axis xyz="0 1 0" />
         <limit effort="${motor_torque}" lower="${-0.25*pi}" upper="${0.25*pi}" velocity="${motor_vec}"/>
-        <dynamics damping="5" friction="10.0" />
+        <dynamics damping="0.5" friction="0.1" />
         <origin xyz="0 0 0.15" rpy="0 0 0" />
         <parent link="torso_yaw_link" />
@@ -114,5 +114,5 @@
         <axis xyz="1 0 0" />
         <limit effort="${motor_torque}" lower="${-0.25*pi}" upper="${0.25*pi}" velocity="${motor_vec}"/>
-        <dynamics damping="5" friction="10" />
+        <dynamics damping="0.5" friction="0.1" />
         <origin xyz="0 0 0" rpy="0 0 0" />
         <parent link="torso_pitch_link" />
@@ -121,5 +121,5 @@
     <link name="torso_link">
         <inertial>
-            <mass value="2" />
+            <mass value="1" />
             <inertia ixx="4.16666667e-06" ixy="0.0" ixz="0.0" iyy="6.6666666667e-6" iyz="0.0" izz="04.16666667e-06" />
         </inertial>
